Commit message: e

File: models/rotors_description/urdf/component_snippets.xacro (robot description, xacro)
@@ -273,81 +273,4 @@
             <zero_position_armed>0</zero_position_armed>
             <joint_control_type>position</joint_control_type>
-          </channel>
-        </control_channels>
-      </plugin>
-    </gazebo>
-  </xacro:macro>
-  <!-- Macro to add the mavlink interface for a fixed-wing model. -->
-  <xacro:macro name="mavlink_interface_macro_fw" params="namespace imu_sub_topic gps_sub_topic mag_sub_topic baro_sub_topic mavlink_addr mavlink_udp_port mavlink_tcp_port serial_enabled serial_device baudrate qgc_addr qgc_udp_port sdk_addr sdk_udp_port hil_mode hil_state_level vehicle_is_tailsitter send_vision_estimation send_odometry enable_lockstep use_tcp">
-    <gazebo>
-      <plugin name="mavlink_interface" filename="libgazebo_mavlink_interface.so">
-        <robotNamespace>${namespace}</robotNamespace>
-        <imuSubTopic>${imu_sub_topic}</imuSubTopic>
-        <gpsSubTopic>${gps_sub_topic}</gpsSubTopic>
-        <magSubTopic>${mag_sub_topic}</magSubTopic>
-        <baroSubTopic>${baro_sub_topic}</baroSubTopic>
-        <mavlink_addr>$(arg mavlink_addr)</mavlink_addr>
-        <mavlink_udp_port>$(arg mavlink_udp_port)</mavlink_udp_port>
-        <mavlink_tcp_port>$(arg mavlink_tcp_port)</mavlink_tcp_port>
-        <serialEnabled>$(arg serial_enabled)</serialEnabled>
-        <serialDevice>$(arg serial_device)</serialDevice>
-        <baudRate>$(arg baudrate)</baudRate>
-        <qgc_addr>$(arg qgc_addr)</qgc_addr>
-        <qgc_udp_port>$(arg qgc_udp_port)</qgc_udp_port>
-        <sdk_addr>$(arg sdk_addr)</sdk_addr>
-        <sdk_udp_port>$(arg sdk_udp_port)</sdk_udp_port>
-        <hil_mode>$(arg hil_mode)</hil_mode>
-        <hil_state_level>$(arg hil_state_level)</hil_state_level>
-        <vehicle_is_tailsitter>$(arg vehicle_is_tailsitter)</vehicle_is_tailsitter>
-        <send_vision_estimation>$(arg send_vision_estimation)</send_vision_estimation>
-        <send_odometry>$(arg send_odometry)</send_odometry>
-        <enable_lockstep>$(arg enable_lockstep)</enable_lockstep>
-        <use_tcp>$(arg use_tcp)</use_tcp>
-        <motorSpeedCommandPubTopic>/gazebo/command/motor_speed</motorSpeedCommandPubTopic>
-        <control_channels>
-          <channel name="rudder">
-            <input_index>2</input_index>
-            <input_offset>0</input_offset>
-            <input_scaling>1</input_scaling>
-            <zero_position_disarmed>0</zero_position_disarmed>
-            <zero_position_armed>0</zero_position_armed>
-            <joint_control_type>position_kinematic</joint_control_type>
-            <joint_name>rudder_joint</joint_name>
-          </channel>
-          <channel name="rotor_4">
-            <input_index>4</input_index>
-            <input_offset>0</input_offset>
-            <input_scaling>3500</input_scaling>
-            <zero_position_disarmed>0</zero_position_disarmed>
-            <zero_position_armed>0</zero_position_armed>
-            <joint_control_type>velocity</joint_control_type>
-            <joint_name>rotor_4_joint</joint_name>
-          </channel>
-          <channel name="left_aileron">
-            <input_index>5</input_index>
-            <input_offset>0</input_offset>
-            <input_scaling>1</input_scaling>
-            <zero_position_disarmed>0</zero_position_disarmed>
-            <zero_position_armed>0</zero_position_armed>
-            <joint_control_type>position_kinematic</joint_control_type>
-            <joint_name>left_elevon_joint</joint_name>
-          </channel>
-          <channel name="right_aileron">
-            <input_index>6</input_index>
-            <input_offset>0</input_offset>
-            <input_scaling>1</input_scaling>
-            <zero_position_disarmed>0</zero_position_disarmed>
-            <zero_position_armed>0</zero_position_armed>
-            <joint_control_type>position_kinematic</joint_control_type>
-            <joint_name>right_elevon_joint</joint_name>
-          </channel>
-          <channel name="elevator">
-            <input_index>7</input_index>
-            <input_offset>0</input_offset>
-            <input_scaling>1</input_scaling>
-            <zero_position_disarmed>0</zero_position_disarmed>
-            <zero_position_armed>0</zero_position_armed>
-            <joint_control_type>position_kinematic</joint_control_type>
-            <joint_name>elevator_joint</joint_name>
           </channel>
         </control_channels>

File: models/rotors_description/urdf/iris_base.xacro (robot description, xacro)
@@ -103,9 +103,9 @@
     imu_topic="/imu"
     mass_imu_sensor="0.015"
-    gyroscope_noise_density="0.00018665"
+    gyroscope_noise_density="0.0003394"
     gyroscopoe_random_walk="0.000038785"
     gyroscope_bias_correlation_time="1000.0"
     gyroscope_turn_on_bias_sigma="0.0087"
-    accelerometer_noise_density="0.00186"
+    accelerometer_noise_density="0.004"
     accelerometer_random_walk="0.006"
     accelerometer_bias_correlation_time="300.0"
